File: adapter/adapter.kicad_pcb (KiCad board)
At the start: 2 copper layers, 93.5 x 50.9 mm, 64 parts, among them J1 RJ9, J10 Ribbon, J11 Ribbon, J12 Ribbon, J13 serial, J14 serial, J2 RJ9, J3 battery charge, J4 RGB, J5 RGB, J6 battery charge, J7 trackball, J8 trackball, J9 Ribbon, SW1 SW_SPST, SW2 SW_SPST, SW3 SW_SPDT, SW4 SW_SPDT, U1 eliteC, U2 eliteC

Commit message: initial work
Parts:
- removed J13, J14: serial, Library:PinHeader_1x04_P2.54mm_Vertical
- removed R5, R6: 5.1k, Library:R_1206_handsolder
- moved J3 40.7 mm to (121.7, 112.5)
- moved R4 12.7 mm to (120.2, 98.4)
- moved R2 12.6 mm to (123.1, 98.4)
- moved J1 12.2 mm to (117.9, 72.9)
- moved J4 10.0 mm to (121.9, 102.9)
- moved J7 4.58 mm to (125.7, 102.9)
- moved J9 2.47 mm to (130.3, 102.9)
- moved J10 1.93 mm to (134.6, 102.8)
Routing:
- net +5V: track 46.5 -> 1.71 mm
- net row2_l: track 37.1 -> 7.27 mm
- net col1_l: track 36.7 -> 7.81 mm
- net col2_l: track 36.0 -> 8.14 mm
- net split_hand_l: track 26.5 -> 0.00 mm, vias 2 -> 0
- net miso_l: track 24.0 -> 0.00 mm
- net sc_l: track 23.7 -> 0.00 mm
- net sda_l: track 38.7 -> 17.9 mm, vias 1 -> 0
- net serial_l: track 22.1 -> 1.93 mm
- net row5_l: track 25.0 -> 5.80 mm
- net scl_l: track 36.2 -> 17.4 mm, vias 2 -> 0
- net col6_l: track 25.1 -> 6.48 mm
- net row1_l: track 34.9 -> 16.3 mm
- net col3_l: track 18.2 -> 0.00 mm
- net col5_l: track 25.1 -> 6.95 mm
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