File: adapter/adapter.kicad_sch (KiCad schematic)
At the start: 30 parts, among them J1 RJ9, J10 Ribbon, J11 Ribbon, J12 Ribbon, J2 RJ9, J3 battery charge, J4 RGB, J5 RGB, J6 battery charge, J7 trackball, J8 trackball, J9 Ribbon, SW1 SW_SPST, SW2 SW_SPST, SW3 SW_SPDT, SW4 SW_SPDT, U1 eliteC, U2 eliteC

Commit message: initial work
Parts:
- removed R5, R6: 5.1k, Library:R_1206_handsolder, symbol Device:R
Changed lines of the file:
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@@
-    (stroke (width 0) (type default))
-  )
-  (wire (pts (xy 261.112 40.513) (xy 261.112 43.688))
     (stroke (width 0) (type default))
   )
@@
   (wire (pts (xy 225.298 44.831) (xy 225.298 46.736))
     (stroke (width 0) (type solid))
-  )
-  (wire (pts (xy 246.253 120.523) (xy 246.253 121.793))
-    (stroke (width 0) (type default))
   )
   (wire (pts (xy 225.298 35.306) (xy 225.298 37.211))
@@
     )
   )
-  (global_label "split_hand_l" (shape input) (at 261.112 43.688 270)
-    (effects (font (size 1.27 1.27)) (justify right))
-    (property "Intersheetrefs" "${INTERSHEET_REFS}" (at 261.1914 55.8378 90)
-      (effects (font (size 1.27 1.27)) (justify right) hide)
-    )
-  )
   (global_label "miso_r" (shape input) (at 133.35 113.03 180)
     (effects (font (size 1.27 1.27)) (justify right))
@@
     (property "Intersheetrefs" "${INTERSHEET_REFS}" (at -1.27 71.12 0)
       (effects (font (size 1.27 1.27)) hide)
-    )
-  )
-  (global_label "split_hand_r" (shape input) (at 246.253 120.523 90)
-    (effects (font (size 1.27 1.27)) (justify left))
-    (property "Intersheetrefs" "${INTERSHEET_REFS}" (at 246.1736 108.3732 90)
-      (effects (font (size 1.27 1.27)) (justify left) hide)
     )
   )
@@
     )
   )
-  (symbol (lib_id "Device:R") (at 246.253 125.603 0) (unit 1)
-    (in_bom yes) (on_board yes) (dnp no)
-    (property "Reference" "R5" (at 248.793 124.333 0)
-      (effects (font (size 1.27 1.27)) (justify left))
-    )
-    (property "Value" "5.1k" (at 248.793 126.873 0)
-      (effects (font (size 1.27 1.27)) (justify left))
-    )
-    (property "Footprint" "Library:R_1206_handsolder" (at 244.475 125.603 90)
-      (effects (font (size 1.27 1.27)) hide)
-    )
-    (property "Datasheet" "~" (at 246.253 125.603 0)
-      (effects (font (size 1.27 1.27)) hide)
-    )
-    (property "JLCPCB BOM" "1" (at 246.253 125.603 0)
-      (effects (font (size 1.27 1.27)) hide)
-    )
-    (property "JLCPCB Part" "C26033" (at 246.253 125.603 0)
-      (effects (font (size 1.27 1.27)) hide)
-    )
-    (pin "1")
-    (pin "2")
-    (instances
-      (project "adapter"
-        (path "/e63e39d7-6ac0-4ffd-8aa3-1841a4541b55"
-          (reference "R5") (unit 1)
-        )
-      )
-    )
-  )
   (symbol (lib_id "power:GND") (at 100.33 110.49 90) (unit 1)
     (in_bom yes) (on_board yes) (dnp no)
@@
     )
   )
-  (symbol (lib_id "Device:R") (at 261.112 36.703 0) (unit 1)
-    (in_bom yes) (on_board yes) (dnp no)
-    (property "Reference" "R6" (at 263.652 35.433 0)
-      (effects (font (size 1.27 1.27)) (justify left))
-    )
-    (property "Value" "5.1k" (at 263.652 37.973 0)
-      (effects (font (size 1.27 1.27)) (justify left))
-    )
-    (property "Footprint" "Library:R_1206_handsolder" (at 259.334 36.703 90)
-      (effects (font (size 1.27 1.27)) hide)
-    )
-    (property "Datasheet" "~" (at 261.112 36.703 0)
-      (effects (font (size 1.27 1.27)) hide)
-    )
-    (property "JLCPCB BOM" "1" (at 261.112 36.703 0)
-      (effects (font (size 1.27 1.27)) hide)
-    )
-    (property "JLCPCB Part" "C26033" (at 261.112 36.703 0)
-      (effects (font (size 1.27 1.27)) hide)
-    )
-    (pin "1")
-    (pin "2")
-    (instances
-      (project "adapter"
-        (path "/e63e39d7-6ac0-4ffd-8aa3-1841a4541b55"
-          (reference "R6") (unit 1)
-        )
-      )
-    )
-  )
   (symbol (lib_id "power:GND") (at 154.432 38.862 270) (unit 1)
     (in_bom yes) (on_board yes) (dnp no)
@@
         (path "/e63e39d7-6ac0-4ffd-8aa3-1841a4541b55"
           (reference "H1") (unit 1)
-        )
-      )
-    )
-  )
-  (symbol (lib_id "power:GND") (at 246.253 129.413 0) (unit 1)
-    (in_bom yes) (on_board yes) (dnp no)
-    (property "Reference" "#PWR0137" (at 246.253 135.763 0)
-      (effects (font (size 1.27 1.27)) hide)
-    )
-    (property "Value" "GND" (at 245.774 132.588 0)
-      (effects (font (size 1.27 1.27)) (justify right))
-    )
-    (property "Footprint" "" (at 246.253 129.413 0)
-      (effects (font (size 1.27 1.27)) hide)
-    )
-    (property "Datasheet" "" (at 246.253 129.413 0)
-      (effects (font (size 1.27 1.27)) hide)
-    )
-    (pin "1")
-    (instances
-      (project "adapter"
-        (path "/e63e39d7-6ac0-4ffd-8aa3-1841a4541b55"
-          (reference "#PWR0137") (unit 1)
         )
       )
@@
         )
       )
-    )
-  )
-  (symbol (lib_id "power:+5V") (at 261.112 32.893 0) (unit 1)
-    (in_bom yes) (on_board yes) (dnp no)
-    (property "Reference" "#PWR0138" (at 261.112 36.703 0)
-      (effects (font (size 1.27 1.27)) hide)
-    )
-    (property "Value" "+5V" (at 262.509 32.131 0)
-      (effects (font (size 1.27 1.27)) (justify left))
-    )
-    (property "Footprint" "" (at 261.112 32.893 0)
-      (effects (font (size 1.27 1.27)) hide)
-    )
-    (property "Datasheet" "" (at 261.112 32.893 0)
-      (effects (font (size 1.27 1.27)) hide)
-    )
-    (pin "1")
-    (instances
-      (project "adapter"
-        (path "/e63e39d7-6ac0-4ffd-8aa3-1841a4541b55"
-          (reference "#PWR0138") (unit 1)
-        )
-      )
